Commit message: Update model

File: model/partial_kitchen/partial_kitchen.urdf (robot description, URDF)
Before this commit: robot iai_dishwasher, 9 links, 8 joints
Joints:
- joint sink_area_left_joint: origin xyz=1.565 1.35 0.35 rpy=0 0 -3.14 -> xyz=1.565 1.35 0.395 rpy=0 0 -3.14
- joint sink_area_right_joint: origin xyz=1.565 -0.782 0.37 rpy=0 0 -3.14 -> xyz=1.565 -0.782 0.395 rpy=0 0 -3.14
- joint sink_area_top_joint: origin xyz=1.565 0.3 0.8 rpy=0 0 -3.14 -> xyz=1.565 0.3 0.825 rpy=0 0 -3.14

Commit message: Add dishwasher model

File: model/partial_kitchen/partial_kitchen.urdf (robot description, URDF)
Before this commit: robot iai_dishwasher, 9 links, 8 joints
Links:
- link sink_area_dish_washer_door_handle: geometry collision box size=0.0164 0.0152 0.5; visual mesh filename=package://iai_kitchen/meshes/handles/Handle60.dae
